Commit message: update

File: src/daedalus_description/urdf/BACKUP/daedalus.xacro (robot description, xacro)
@@ -2,5 +2,5 @@
 <robot name="daedalus"
  xmlns:xacro="http://www.ros.org/wiki/xacro">
-	<xacro:property name="const" value="0.1" />
+	<xacro:property name="const" value="0.01" />
   <gazebo>
     <plugin name="gazebo_ros_control" filename="libgazebo_ros_control.so">
@@ -12,11 +12,11 @@
 	<inertial>
         <origin xyz="0 0 0" rpy="0 0 0"/>
-          <mass value="${240.264202 * const}"/>
-        <inertia ixx="0.01" ixy="0" ixz="0" iyy="0.01" iyz="0" izz="0.01"/>
+          <mass value="${24.264202 * const}"/>
+        <inertia ixx="10" ixy="0" ixz="0" iyy="10" iyz="0" izz="10"/>
       </inertial>
       <visual>
 	  	<origin xyz="0 0 0" rpy="0 0 0" />
 		<geometry>
-			<box size="0.25 0.15 0.05" />
+			<box size="0.2 0.3 0.05" />
 		</geometry>
       </visual>
@@ -27,15 +27,15 @@
 		<material>Gazebo/Black</material>
 	</gazebo>
-	<leg flipped="1" parent="frame" suffix="1">
-		<origin rpy="0 0 3.14" xyz="0.125 0.075 0"/>
+	<leg parent="frame" suffix="1">
+		<origin rpy="0 0 3.14" xyz="0.15 0.15 0"/>
 	</leg>
-	<leg flipped="0" parent="frame" suffix="2">
-		<origin rpy="0 0 3.14" xyz="0.125 -0.075 0"/>
+	<leg parent="frame" suffix="2">
+		<origin rpy="0 0 0" xyz="0.15 -0.15 0"/>
 	</leg>
-	<leg flipped="0" parent="frame" suffix="3">
-		<origin rpy="0 0 0" xyz="-0.125 0.075 0"/>
+	<leg parent="frame" suffix="3">
+		<origin rpy="0 0 0" xyz="-0.15 0.15 0"/>
 	</leg>
-	<leg flipped="1" parent="frame" suffix="4">
-		<origin rpy="0 0 0" xyz="-0.125 -0.075 0"/>
+	<leg parent="frame" suffix="4">
+		<origin rpy="0 0 3.14" xyz="-0.15 -0.15 0"/>
 	</leg>
 </robot>

File: src/daedalus_description/urdf/BACKUP/leg _OLD.xacro (robot description, xacro)
@@ -1,15 +1,11 @@
 <?xml version="1.0"?>
 <robot xmlns:xacro="http://www.ros.org/wiki/xacro">
-	<xacro:include filename="$(find daedalus_description)/urdf/daedalus.gazebo" />
-	<xacro:include filename="$(find daedalus_description)/urdf/materials.xacro" />
-	<xacro:property name="scale" value="0.01" />
-	<macro name="leg" params="suffix parent flipped *origin">
+	<macro name="leg" params="suffix parent *origin">
 	<leg_finish suffix="${suffix}"/>
     <link name="leg${suffix}link0">
-    	<self_collide>1</self_collide>
       <inertial>
         <origin xyz="0 0 0" rpy="0 0 0"/>
-          <mass value="${47.264202 * const}"/>
-        <inertia ixx="${92.924561*scale}" ixy="0" ixz="0" iyy="${112.408630*scale}" iyz="0" izz="${106.058662*scale}"/>
+          <mass value="${4.72639954 * const}"/>
+        <inertia ixx="3.76702192" ixy="0" ixz="0" iyy="5.02939053" iyz="0" izz="0.104767786"/>
       </inertial>
       <collision name="collision">
@@ -27,12 +23,11 @@
     </link>
     <link name="leg${suffix}link1">
-    	<self_collide>1</self_collide>
-      <inertial>
-        <origin xyz="-0.0236 0 0" rpy="0 0 0"/>
-        <mass value="${62.343552 * const}"/>
-        <inertia ixx="${256.757294*scale}" ixy="${0.461719*scale}" ixz="${40.230606*scale}" iyy="${280.351624*scale}" iyz="${-1.692201*scale}" izz="${114.922241*scale}"/>
-      </inertial>
-      <collision name="collision">
-        <origin xyz="-0.0236 0 0" rpy="0 0 0"/>
+      <inertial>
+        <origin xyz="0.837170246 1.0317214 0.161524277" rpy="0 0 0"/>
+        <mass value="${6.23121787 * const}"/>
+        <inertia ixx="4.36786663" ixy="0" ixz="0" iyy="6.63326988" iyz="0" izz="0.164683289"/>
+      </inertial>
+      <collision name="collision">
+        <origin xyz="-0.86 -1.03 -0.17" rpy="0 0 0"/>
         <geometry>
           <mesh filename="package://daedalus_description/meshes/link1.dae"/>
@@ -40,5 +35,5 @@
       </collision>
       <visual name="visual">
-        <origin xyz="-0.0236 0 0" rpy="0 0 0"/>
+        <origin xyz="-0.86 -1.03 -0.17" rpy="0 0 0"/>
         <geometry>
           <mesh filename="package://daedalus_description/meshes/link1.dae"/>
@@ -49,10 +44,10 @@
       <self_collide>1</self_collide>
       <inertial>
-        <origin xyz="0 0.0371 -0.0015" rpy="0 0 0"/>
-        <mass value="${73.212067 * const}"/>
-        <inertia ixx="${308.272949*scale}" ixy="0" ixz="0" iyy="${141.348206*scale}" iyz="${-6.197227*scale}" izz="${320.700867*scale}"/>
-      </inertial>
-      <collision name="collision">
-        <origin xyz="0 0.0371 -0.0015" rpy="0 0 0"/>
+        <origin xyz="-0.017799314 0.04493617  -0.002242117" rpy="0 0 0"/>
+        <mass value="${7.32147232 * const}"/>
+        <inertia ixx="5.071313" ixy="0" ixz="0" iyy="8.46231008" iyz="0" izz="0.316663829"/>
+      </inertial>
+      <collision name="collision">
+        <origin xyz="-0.85 -1.03 -0.21" rpy="0 0 0"/>
         <geometry>
           <mesh filename="package://daedalus_description/meshes/link2.dae"/>
@@ -60,5 +55,5 @@
       </collision>
       <visual name="visual">
-        <origin xyz="0 0.0371 -0.0015" rpy="0 0 0"/>
+        <origin xyz="-0.85 -1.03 -0.21" rpy="0 0 0"/>
         <geometry>
           <mesh filename="package://daedalus_description/meshes/link2.dae"/>
@@ -69,10 +64,10 @@
       <self_collide>1</self_collide>
       <inertial>
-        <origin xyz=" 0 -0.0041 -0.0371" rpy="0 0 0"/>
-        <mass value="${43.109013  * const}"/>
-        <inertia ixx="${177.687561*scale}" ixy="0" ixz="0" iyy="${208.616043*scale}" iyz="${-14.718610*scale}" izz="${59.618698*scale}"/>
-      </inertial>
-      <collision name="collision">
-        <origin xyz="0 -0.0041 -0.0371" rpy="0 0 0"/>
+        <origin xyz=" -0.0177993  -0.0027828  -0.0402923" rpy="0 0 0"/>
+        <mass value="${4.31132052  * const}"/>
+        <inertia ixx="2.98629222" ixy="0" ixz="0" iyy="5.09630234" iyz="0" izz="0.0982604921"/>
+      </inertial>
+      <collision name="collision">
+        <origin xyz="-0.85 -1.09 -0.19" rpy="0 0 0"/>
         <geometry>
           <mesh filename="package://daedalus_description/meshes/link3.dae"/>
@@ -80,5 +75,5 @@
       </collision>
       <visual name="visual">
-        <origin xyz="0 -0.0041 -0.0371" rpy="0 0 0"/>
+        <origin xyz="-0.85 -1.09 -0.19" rpy="0 0 0"/>
         <geometry>
           <mesh filename="package://daedalus_description/meshes/link3.dae"/>
@@ -89,10 +84,10 @@
       <self_collide>1</self_collide>
       <inertial>
-        <origin xyz="0.0002  -0.0233 -0.0124" rpy="0 0 0"/>
-        <mass value="${79.043472 * const}"/>
-        <inertia ixx="${609.197083*scale}" ixy="${13.511174*scale}" ixz="${-5.220560*scale}" iyy="${234.447556*scale}" iyz="${179.840118*scale}" izz="${511.354614*scale}"/>
-      </inertial>
-      <collision name="collision">
-        <origin xyz="0.0002  -0.0233 -0.0124" rpy="0 0 0"/>
+        <origin xyz="0.0230260  -0.0192363  -0.0096265" rpy="0 0 0"/>
+        <mass value="${7.90197358 * const}"/>
+        <inertia ixx="5.48411837" ixy="0" ixz="0" iyy="8.72903423" iyz="0" izz="0.0812723132"/>
+      </inertial>
+      <collision name="collision">
+        <origin xyz="-0.81 -1.07 -0.11" rpy="0 0 0"/>
         <geometry>
           <mesh filename="package://daedalus_description/meshes/link4.dae"/>
@@ -100,5 +95,5 @@
       </collision>
       <visual name="visual">
-        <origin xyz="0.0002  -0.0233 -0.0124" rpy="0 0 0"/>
+        <origin xyz="-0.81 -1.07 -0.11" rpy="0 0 0"/>
         <geometry>
           <mesh filename="package://daedalus_description/meshes/link4.dae"/>
@@ -109,10 +104,10 @@
       <self_collide>1</self_collide>
       <inertial>
-        <origin xyz="-0.0006 -0.0009 -0.0311" rpy="0 0 0"/>
-        <mass value="${65.552696 * const}"/>
-        <inertia ixx="${385.638153*scale}" ixy="${-0.223889*scale}" ixz="${-13.452513*scale}" iyy="${286.320038*scale}" iyz="${-3.575976*scale}" izz="${338.489807*scale}"/>
-      </inertial>
-      <collision name="collision">
-        <origin xyz="-0.0006 -0.0009 -0.0311" rpy="0 0 0"/>
+        <origin xyz="0.0019165   0.0104236  -0.0496145" rpy="0 0 0"/>
+        <mass value="${6.55679875 * const}"/>
+        <inertia ixx="4.53905844" ixy="0" ixz="0" iyy="7.09980012" iyz="0" izz="0.012361989"/>
+      </inertial>
+      <collision name="collision">
+        <origin xyz="-0.83 -1.03 -0.09" rpy="0 0 0"/>
         <geometry>
           <mesh filename="package://daedalus_description/meshes/link5.dae"/>
@@ -120,5 +115,5 @@
       </collision>
       <visual name="visual">
-        <origin xyz="-0.0006 -0.0009 -0.0311" rpy="0 0 0"/>
+        <origin xyz="-0.83 -1.03 -0.09" rpy="0 0 0"/>
         <geometry>
           <mesh filename="package://daedalus_description/meshes/link5.dae"/>
@@ -133,37 +128,37 @@
     </joint>
     <joint type="revolute" name="leg${suffix}joint1">
-      <origin xyz="-0.0249 0 0.0205" rpy="0 0 0"/>
+      <origin xyz="0 0 0" rpy="0 0 0"/>
       <child link="leg${suffix}link1"/>
       <parent link="leg${suffix}link0"/>"
-      <axis xyz="0 0 -1"/>
-      <limit lower="-1.57" upper="1.57" effort="100" velocity="10"/>
+      <axis xyz="0 0 1"/>
+      <limit lower="-1.57" upper="1.57" effort="100" velocity="0.5"/>
     </joint>
     <joint type="revolute" name="leg${suffix}joint2">
-      <origin xyz="-0.0309 0.0002 0.0381" rpy="${3.14159/2} 0 ${3.14159 * flipped}"/>
+      <origin xyz="-0.01 0 0.04" rpy="0 0 0"/>
       <child link="leg${suffix}link2"/>
       <parent link="leg${suffix}link1"/>
-      <axis xyz="${1 - 2 * flipped} 0 0"/>
-      <limit lower="-1.57" upper="1.57" effort="100" velocity="10"/>
+      <axis xyz="1 0 0"/>
+      <limit lower="-0.45" upper="3.59" effort="100" velocity="0.5"/>
     </joint>
     <joint type="revolute" name="leg${suffix}joint3">
-      <origin xyz="0 0.0564 -0.0208" rpy="0 0 0"/>
+      <origin xyz="0 0.06 -0.02" rpy="0 0 0"/>
       <child link="leg${suffix}link3"/>
       <parent link="leg${suffix}link2"/>
-      <axis xyz="${2 * flipped - 1} 0 0"/>
-      <limit lower="-1.57" upper="1.57" effort="100" velocity="10"/>
+      <axis xyz="1 0 0"/>
+      <limit lower="-1.57" upper="1.57" effort="100" velocity="0.5"/>
     </joint>
     <joint type="revolute" name="leg${suffix}joint4">
-      <origin xyz="0 -0.0171 -0.0742" rpy="${-3.14159/4} 0 0"/>
+      <origin xyz="-0.04 -0.02 -0.08" rpy="0 0 0"/>
       <child link="leg${suffix}link4"/>
       <parent link="leg${suffix}link3"/>
-      <axis xyz="${2 * flipped - 1} 0 0"/>
-      <limit lower="-1.57" upper="1.57" effort="100" velocity="10"/>
+      <axis xyz="1 0 0"/>
+      <limit lower="-1.57" upper="1.57" effort="100" velocity="0.5"/>
     </joint>
     <joint type="revolute" name="leg${suffix}joint5">
-      <origin xyz="-0.0004 -0.0411 -0.0248" rpy="0 0 0"/>
+      <origin xyz="0.02 -0.04 -0.02" rpy="0 0 0"/>
       <child link="leg${suffix}link5"/>
       <parent link="leg${suffix}link4"/>
       <axis xyz="0 1 0"/>
-      <limit lower="-1.57" upper="1.57" effort="100" velocity="10"/>
+      <limit lower="-1.57" upper="1.57" effort="100" velocity="0.5"/>
     </joint>
 <transmission name="tran1">

File: src/daedalus_description/urdf/BACKUP/leg.xacro (robot description, xacro)
@@ -4,5 +4,5 @@
 	<xacro:include filename="$(find daedalus_description)/urdf/materials.xacro" />
 	<xacro:property name="scale" value="0.01" />
-	<macro name="leg" params="suffix parent flipped *origin">
+	<macro name="leg" params="suffix parent *origin">
 	<leg_finish suffix="${suffix}"/>
     <link name="leg${suffix}link0">
@@ -29,10 +29,10 @@
     	<self_collide>1</self_collide>
       <inertial>
-        <origin xyz="-0.0236 0 0" rpy="0 0 0"/>
+        <origin xyz="0.837170246 1.0317214 0.161524277" rpy="0 0 0"/>
         <mass value="${62.343552 * const}"/>
         <inertia ixx="${256.757294*scale}" ixy="${0.461719*scale}" ixz="${40.230606*scale}" iyy="${280.351624*scale}" iyz="${-1.692201*scale}" izz="${114.922241*scale}"/>
       </inertial>
       <collision name="collision">
-        <origin xyz="-0.0236 0 0" rpy="0 0 0"/>
+        <origin xyz="-0.86 -1.03 -0.17" rpy="0 0 0"/>
         <geometry>
           <mesh filename="package://daedalus_description/meshes/link1.dae"/>
@@ -40,5 +40,5 @@
       </collision>
       <visual name="visual">
-        <origin xyz="-0.0236 0 0" rpy="0 0 0"/>
+        <origin xyz="-0.86 -1.03 -0.17" rpy="0 0 0"/>
         <geometry>
           <mesh filename="package://daedalus_description/meshes/link1.dae"/>
@@ -49,10 +49,10 @@
       <self_collide>1</self_collide>
       <inertial>
-        <origin xyz="0 0.0371 -0.0015" rpy="0 0 0"/>
+        <origin xyz="-0.017799314 0.04493617  -0.002242117" rpy="0 0 0"/>
         <mass value="${73.212067 * const}"/>
         <inertia ixx="${308.272949*scale}" ixy="0" ixz="0" iyy="${141.348206*scale}" iyz="${-6.197227*scale}" izz="${320.700867*scale}"/>
       </inertial>
       <collision name="collision">
-        <origin xyz="0 0.0371 -0.0015" rpy="0 0 0"/>
+        <origin xyz="-0.85 -1.03 -0.21" rpy="0 0 0"/>
         <geometry>
           <mesh filename="package://daedalus_description/meshes/link2.dae"/>
@@ -60,5 +60,5 @@
       </collision>
       <visual name="visual">
-        <origin xyz="0 0.0371 -0.0015" rpy="0 0 0"/>
+        <origin xyz="-0.85 -1.03 -0.21" rpy="0 0 0"/>
         <geometry>
           <mesh filename="package://daedalus_description/meshes/link2.dae"/>
@@ -69,10 +69,10 @@
       <self_collide>1</self_collide>
       <inertial>
-        <origin xyz=" 0 -0.0041 -0.0371" rpy="0 0 0"/>
+        <origin xyz=" -0.0177993  -0.0027828  -0.0402923" rpy="0 0 0"/>
         <mass value="${43.109013  * const}"/>
         <inertia ixx="${177.687561*scale}" ixy="0" ixz="0" iyy="${208.616043*scale}" iyz="${-14.718610*scale}" izz="${59.618698*scale}"/>
       </inertial>
       <collision name="collision">
-        <origin xyz="0 -0.0041 -0.0371" rpy="0 0 0"/>
+        <origin xyz="-0.85 -1.09 -0.19" rpy="0 0 0"/>
         <geometry>
           <mesh filename="package://daedalus_description/meshes/link3.dae"/>
@@ -80,5 +80,5 @@
       </collision>
       <visual name="visual">
-        <origin xyz="0 -0.0041 -0.0371" rpy="0 0 0"/>
+        <origin xyz="-0.85 -1.09 -0.19" rpy="0 0 0"/>
         <geometry>
           <mesh filename="package://daedalus_description/meshes/link3.dae"/>
@@ -89,10 +89,10 @@
       <self_collide>1</self_collide>
       <inertial>
-        <origin xyz="0.0002  -0.0233 -0.0124" rpy="0 0 0"/>
+        <origin xyz="0.0230260  -0.0192363  -0.0096265" rpy="0 0 0"/>
         <mass value="${79.043472 * const}"/>
         <inertia ixx="${609.197083*scale}" ixy="${13.511174*scale}" ixz="${-5.220560*scale}" iyy="${234.447556*scale}" iyz="${179.840118*scale}" izz="${511.354614*scale}"/>
       </inertial>
       <collision name="collision">
-        <origin xyz="0.0002  -0.0233 -0.0124" rpy="0 0 0"/>
+        <origin xyz="-0.81 -1.07 -0.11" rpy="0 0 0"/>
         <geometry>
           <mesh filename="package://daedalus_description/meshes/link4.dae"/>
@@ -100,5 +100,5 @@
       </collision>
       <visual name="visual">
-        <origin xyz="0.0002  -0.0233 -0.0124" rpy="0 0 0"/>
+        <origin xyz="-0.81 -1.07 -0.11" rpy="0 0 0"/>
         <geometry>
           <mesh filename="package://daedalus_description/meshes/link4.dae"/>
@@ -109,10 +109,10 @@
       <self_collide>1</self_collide>
       <inertial>
-        <origin xyz="-0.0006 -0.0009 -0.0311" rpy="0 0 0"/>
+        <origin xyz="0.0019165   0.0104236  -0.0496145" rpy="0 0 0"/>
         <mass value="${65.552696 * const}"/>
         <inertia ixx="${385.638153*scale}" ixy="${-0.223889*scale}" ixz="${-13.452513*scale}" iyy="${286.320038*scale}" iyz="${-3.575976*scale}" izz="${338.489807*scale}"/>
       </inertial>
       <collision name="collision">
-        <origin xyz="-0.0006 -0.0009 -0.0311" rpy="0 0 0"/>
+        <origin xyz="-0.83 -1.03 -0.09" rpy="0 0 0"/>
         <geometry>
           <mesh filename="package://daedalus_description/meshes/link5.dae"/>
@@ -120,5 +120,5 @@
       </collision>
       <visual name="visual">
-        <origin xyz="-0.0006 -0.0009 -0.0311" rpy="0 0 0"/>
+        <origin xyz="-0.83 -1.03 -0.09" rpy="0 0 0"/>
         <geometry>
           <mesh filename="package://daedalus_description/meshes/link5.dae"/>
@@ -133,37 +133,37 @@
     </joint>
     <joint type="revolute" name="leg${suffix}joint1">
-      <origin xyz="-0.0249 0 0.0205" rpy="0 0 0"/>
+      <origin xyz="0 0 0" rpy="0 0 0"/>
       <child link="leg${suffix}link1"/>
       <parent link="leg${suffix}link0"/>"
-      <axis xyz="0 0 -1"/>
-      <limit lower="-1.57" upper="1.57" effort="100" velocity="10"/>
+      <axis xyz="0 0 1"/>
+      <limit lower="-1.57" upper="1.57" effort="100" velocity="0.5"/>
     </joint>
     <joint type="revolute" name="leg${suffix}joint2">
-      <origin xyz="-0.0309 0.0002 0.0381" rpy="${3.14159/2} 0 ${3.14159 * flipped}"/>
+      <origin xyz="-0.01 0 0.04" rpy="0 0 0"/>
       <child link="leg${suffix}link2"/>
       <parent link="leg${suffix}link1"/>
-      <axis xyz="${1 - 2 * flipped} 0 0"/>
-      <limit lower="-1.57" upper="1.57" effort="100" velocity="10"/>
+      <axis xyz="1 0 0"/>
+      <limit lower="-0.45" upper="3.59" effort="100" velocity="0.5"/>
     </joint>
     <joint type="revolute" name="leg${suffix}joint3">
-      <origin xyz="0 0.0564 -0.0208" rpy="0 0 0"/>
+      <origin xyz="0 0.06 -0.02" rpy="0 0 0"/>
       <child link="leg${suffix}link3"/>
       <parent link="leg${suffix}link2"/>
-      <axis xyz="${2 * flipped - 1} 0 0"/>
-      <limit lower="-1.57" upper="1.57" effort="100" velocity="10"/>
+      <axis xyz="1 0 0"/>
+      <limit lower="-1.57" upper="1.57" effort="100" velocity="0.5"/>
     </joint>
     <joint type="revolute" name="leg${suffix}joint4">
-      <origin xyz="0 -0.0171 -0.0742" rpy="${-3.14159/4} 0 0"/>
+      <origin xyz="-0.04 -0.02 -0.08" rpy="0 0 0"/>
       <child link="leg${suffix}link4"/>
       <parent link="leg${suffix}link3"/>
-      <axis xyz="${2 * flipped - 1} 0 0"/>
-      <limit lower="-1.57" upper="1.57" effort="100" velocity="10"/>
+      <axis xyz="1 0 0"/>
+      <limit lower="-1.57" upper="1.57" effort="100" velocity="0.5"/>
     </joint>
     <joint type="revolute" name="leg${suffix}joint5">
-      <origin xyz="-0.0004 -0.0411 -0.0248" rpy="0 0 0"/>
+      <origin xyz="0.02 -0.04 -0.02" rpy="0 0 0"/>
       <child link="leg${suffix}link5"/>
       <parent link="leg${suffix}link4"/>
       <axis xyz="0 1 0"/>
-      <limit lower="-1.57" upper="1.57" effort="100" velocity="10"/>
+      <limit lower="-1.57" upper="1.57" effort="100" velocity="0.5"/>
     </joint>
 <transmission name="tran1">
