Commit message: some kind of gait/better inertia

File: src/daedalus_description/urdf/daedalus.xacro (robot description, xacro)
@@ -2,5 +2,5 @@
 <robot name="daedalus"
  xmlns:xacro="http://www.ros.org/wiki/xacro">
-	<xacro:property name="const" value="0.1" />
+	<xacro:property name="const" value="0.01" />
   <gazebo>
     <plugin name="gazebo_ros_control" filename="libgazebo_ros_control.so">
@@ -10,20 +10,32 @@
 	<xacro:include filename="$(find daedalus_description)/urdf/leg.xacro" />
   	<link name="frame">
-      <inertial>
+	<inertial>
         <origin xyz="0 0 0" rpy="0 0 0"/>
-		<mass value="${2.72639954 * const}"/>
+          <mass value="${24.264202 * const}"/>
+        <inertia ixx="10" ixy="0" ixz="0" iyy="10" iyz="0" izz="10"/>
       </inertial>
+      <visual>
+	  	<origin xyz="0 0 0" rpy="0 0 0" />
+		<geometry>
+			<box size="0.2 0.3 0.05" />
+		</geometry>
+      </visual>
   	</link>
+  	<gazebo reference="frame">
+		<mu1>0.2</mu1>
+		<mu2>0.2</mu2>
+		<material>Gazebo/Black</material>
+	</gazebo>
 	<leg parent="frame" suffix="1">
-		<origin rpy="0 0 0" xyz="0 0 0"/>
+		<origin rpy="0 0 3.14" xyz="0.15 0.15 0"/>
 	</leg>
 	<leg parent="frame" suffix="2">
-		<origin rpy="0 0 0" xyz="0.3 0 0"/>
+		<origin rpy="0 0 0" xyz="0.15 -0.15 0"/>
 	</leg>
 	<leg parent="frame" suffix="3">
-		<origin rpy="0 0 0" xyz="0 0.3 0"/>
+		<origin rpy="0 0 0" xyz="-0.15 0.15 0"/>
 	</leg>
 	<leg parent="frame" suffix="4">
-		<origin rpy="0 0 0" xyz="0.3 0.3 0"/>
+		<origin rpy="0 0 3.14" xyz="-0.15 -0.15 0"/>
 	</leg>
 </robot>

File: src/daedalus_description/urdf/leg.xacro (robot description, xacro)
@@ -1,10 +1,15 @@
 <?xml version="1.0"?>
 <robot xmlns:xacro="http://www.ros.org/wiki/xacro">
+	<xacro:include filename="$(find daedalus_description)/urdf/daedalus.gazebo" />
+	<xacro:include filename="$(find daedalus_description)/urdf/materials.xacro" />
+	<xacro:property name="scale" value="0.01" />
 	<macro name="leg" params="suffix parent *origin">
+	<leg_finish suffix="${suffix}"/>
     <link name="leg${suffix}link0">
+    	<self_collide>1</self_collide>
       <inertial>
         <origin xyz="0 0 0" rpy="0 0 0"/>
-          <mass value="${4.72639954 * const}"/>
-        <inertia ixx="3.76702192" ixy="0" ixz="0" iyy="5.02939053" iyz="0" izz="0.104767786"/>
+          <mass value="${47.264202 * const}"/>
+        <inertia ixx="${92.924561*scale}" ixy="0" ixz="0" iyy="${112.408630*scale}" iyz="0" izz="${106.058662*scale}"/>
       </inertial>
       <collision name="collision">
@@ -22,8 +27,9 @@
     </link>
     <link name="leg${suffix}link1">
+    	<self_collide>1</self_collide>
       <inertial>
         <origin xyz="0.837170246 1.0317214 0.161524277" rpy="0 0 0"/>
-        <mass value="${6.23121787 * const}"/>
-        <inertia ixx="4.36786663" ixy="0" ixz="0" iyy="6.63326988" iyz="0" izz="0.164683289"/>
+        <mass value="${62.343552 * const}"/>
+        <inertia ixx="${256.757294*scale}" ixy="${0.461719*scale}" ixz="${40.230606*scale}" iyy="${280.351624*scale}" iyz="${-1.692201*scale}" izz="${114.922241*scale}"/>
       </inertial>
       <collision name="collision">
@@ -44,6 +50,6 @@
       <inertial>
         <origin xyz="-0.017799314 0.04493617  -0.002242117" rpy="0 0 0"/>
-        <mass value="${7.32147232 * const}"/>
-        <inertia ixx="5.071313" ixy="0" ixz="0" iyy="8.46231008" iyz="0" izz="0.316663829"/>
+        <mass value="${73.212067 * const}"/>
+        <inertia ixx="${308.272949*scale}" ixy="0" ixz="0" iyy="${141.348206*scale}" iyz="${-6.197227*scale}" izz="${320.700867*scale}"/>
       </inertial>
       <collision name="collision">
@@ -64,6 +70,6 @@
       <inertial>
         <origin xyz=" -0.0177993  -0.0027828  -0.0402923" rpy="0 0 0"/>
-        <mass value="${4.31132052  * const}"/>
-        <inertia ixx="2.98629222" ixy="0" ixz="0" iyy="5.09630234" iyz="0" izz="0.0982604921"/>
+        <mass value="${43.109013  * const}"/>
+        <inertia ixx="${177.687561*scale}" ixy="0" ixz="0" iyy="${208.616043*scale}" iyz="${-14.718610*scale}" izz="${59.618698*scale}"/>
       </inertial>
       <collision name="collision">
@@ -84,6 +90,6 @@
       <inertial>
         <origin xyz="0.0230260  -0.0192363  -0.0096265" rpy="0 0 0"/>
-        <mass value="${7.90197358 * const}"/>
-        <inertia ixx="5.48411837" ixy="0" ixz="0" iyy="8.72903423" iyz="0" izz="0.0812723132"/>
+        <mass value="${79.043472 * const}"/>
+        <inertia ixx="${609.197083*scale}" ixy="${13.511174*scale}" ixz="${-5.220560*scale}" iyy="${234.447556*scale}" iyz="${179.840118*scale}" izz="${511.354614*scale}"/>
       </inertial>
       <collision name="collision">
@@ -104,6 +110,6 @@
       <inertial>
         <origin xyz="0.0019165   0.0104236  -0.0496145" rpy="0 0 0"/>
-        <mass value="${6.55679875 * const}"/>
-        <inertia ixx="4.53905844" ixy="0" ixz="0" iyy="7.09980012" iyz="0" izz="0.012361989"/>
+        <mass value="${65.552696 * const}"/>
+        <inertia ixx="${385.638153*scale}" ixy="${-0.223889*scale}" ixz="${-13.452513*scale}" iyy="${286.320038*scale}" iyz="${-3.575976*scale}" izz="${338.489807*scale}"/>
       </inertial>
       <collision name="collision">

Commit message: update on late Sep.

File: src/daedalus_description/urdf/daedalus.xacro (robot description, xacro)
@@ -2,5 +2,5 @@
 <robot name="daedalus"
  xmlns:xacro="http://www.ros.org/wiki/xacro">
-	<xacro:property name="const" value="0.1" />
+	<xacro:property name="const" value="0.2" />
   <gazebo>
     <plugin name="gazebo_ros_control" filename="libgazebo_ros_control.so">
@@ -9,4 +9,6 @@
   </gazebo>
 	<xacro:include filename="$(find daedalus_description)/urdf/leg.xacro" />
+    <link name="root"/>
+    <virtual_joint name="v_root" type="fixed" parent_frame="world" child_link="root" />
   	<link name="frame">
 	<inertial>
@@ -27,4 +29,8 @@
 		<material>Gazebo/Black</material>
 	</gazebo>
+    <joint type="fixed" name="r_root">
+      <child link="frame"/>
+      <parent link="root"/>
+    </joint>
 	<leg flipped="1" parent="frame" suffix="1">
 		<origin rpy="0 0 3.14" xyz="0.125 0.075 0"/>

Commit message: New Commit on GitLab

File: src/daedalus_description/urdf/daedalus.xacro (robot description, xacro)
@@ -2,10 +2,12 @@
 <robot name="daedalus"
  xmlns:xacro="http://www.ros.org/wiki/xacro">
-	<xacro:property name="const" value="0.2" />
-  <gazebo>
-    <plugin name="gazebo_ros_control" filename="libgazebo_ros_control.so">
-      <robotNamespace>/daedalus</robotNamespace>
-    </plugin>
-  </gazebo>
+	<!--xacro:property name="const" value="0.2" /-->
+	<xacro:property name="const" value="1e-2" />
+	<!-- <xacro:property name="const" value="0.01" /> -->
+	<gazebo>
+	    <plugin name="gazebo_ros_control" filename="libgazebo_ros_control.so">
+	      <robotNamespace>/daedalus</robotNamespace>
+	    </plugin>
+	</gazebo>
 	<xacro:include filename="$(find daedalus_description)/urdf/leg.xacro" />
     <link name="root"/>
@@ -15,16 +17,30 @@
         <origin xyz="0 0 0" rpy="0 0 0"/>
           <mass value="${240.264202 * const}"/>
-        <inertia ixx="0.01" ixy="0" ixz="0" iyy="0.01" iyz="0" izz="0.01"/>
+        <inertia ixx="0.000367" ixy="0" ixz="0" iyy="0.000630" iyz="0" izz="0.000862"/>
+        <!-- <inertia ixx="0" ixy="0" ixz="0" iyy="0" iyz="0" izz="0"/> -->
       </inertial>
+      <collision>
+	  	<origin xyz="0 0 0" rpy="0 0 0" />
+		<geometry>
+			<box size="0.28 0.125 0.06" />
+		</geometry>
+      </collision>
+<!--       <visual name="visual">
+        <origin xyz="0 0 0" rpy="0 0 0"/>
+        <geometry>
+          <mesh filename="package://daedalus_description/meshes/FRAME_new.dae"/>
+        </geometry>
+      </visual>
+ -->
       <visual>
 	  	<origin xyz="0 0 0" rpy="0 0 0" />
 		<geometry>
-			<box size="0.25 0.15 0.05" />
+			<box size="0.28 0.125 0.06" />
 		</geometry>
       </visual>
   	</link>
   	<gazebo reference="frame">
-		<mu1>0.2</mu1>
-		<mu2>0.2</mu2>
+		<!-- <mu1>0.2</mu1>
+		<mu2>0.2</mu2> -->
 		<material>Gazebo/Black</material>
 	</gazebo>
@@ -34,14 +50,14 @@
     </joint>
 	<leg flipped="1" parent="frame" suffix="1">
-		<origin rpy="0 0 3.14" xyz="0.125 0.075 0"/>
+		<origin rpy="0 0 3.14" xyz="0.14 0.0625 0"/>
 	</leg>
 	<leg flipped="0" parent="frame" suffix="2">
-		<origin rpy="0 0 3.14" xyz="0.125 -0.075 0"/>
+		<origin rpy="0 0 3.14" xyz="0.14 -0.0625 0"/>
 	</leg>
 	<leg flipped="0" parent="frame" suffix="3">
-		<origin rpy="0 0 0" xyz="-0.125 0.075 0"/>
+		<origin rpy="0 0 0" xyz="-0.14 0.0625 0"/>
 	</leg>
 	<leg flipped="1" parent="frame" suffix="4">
-		<origin rpy="0 0 0" xyz="-0.125 -0.075 0"/>
+		<origin rpy="0 0 0" xyz="-0.14 -0.0625 0"/>
 	</leg>
 </robot>

File: src/daedalus_description/urdf/leg.xacro (robot description, xacro)
@@ -3,5 +3,19 @@
 	<xacro:include filename="$(find daedalus_description)/urdf/daedalus.gazebo" />
 	<xacro:include filename="$(find daedalus_description)/urdf/materials.xacro" />
-	<xacro:property name="scale" value="0.01" />
+	<!--xacro:property name="scale" value="0.01" /-->
+	<xacro:property name="scale" value="1e-6" />
+	<!--xacro:property name="scale" value="0" /-->
+  <!-- <xacro:property name="m0" value="1" />
+  <xacro:property name="m1" value="1" />
+  <xacro:property name="m2" value="1" />
+  <xacro:property name="m3" value="1" />
+  <xacro:property name="m4" value="1" />
+  <xacro:property name="m5" value="1" /> -->
+  <xacro:property name="m0" value="${47.264202 * const}" />
+  <xacro:property name="m1" value="${62.343552 * const}" />
+  <xacro:property name="m2" value="${73.212067 * const}" />
+  <xacro:property name="m3" value="${43.109013 * const}" />
+  <xacro:property name="m4" value="${79.043472 * const}" />
+  <xacro:property name="m5" value="${65.552696 * const}" />
 	<macro name="leg" params="suffix parent flipped *origin">
 	<leg_finish suffix="${suffix}"/>
@@ -10,6 +24,6 @@
       <inertial>
         <origin xyz="0 0 0" rpy="0 0 0"/>
-          <mass value="${47.264202 * const}"/>
-        <inertia ixx="${92.924561*scale}" ixy="0" ixz="0" iyy="${112.408630*scale}" iyz="0" izz="${106.058662*scale}"/>
+          <mass value="${m0}"/>
+        <inertia ixx="${92.924561*scale*m0}" ixy="0" ixz="0" iyy="${112.408630*scale*m0}" iyz="0" izz="${106.058662*scale*m0}"/>
       </inertial>
       <collision name="collision">
@@ -30,6 +44,6 @@
       <inertial>
         <origin xyz="-0.0236 0 0" rpy="0 0 0"/>
-        <mass value="${62.343552 * const}"/>
-        <inertia ixx="${256.757294*scale}" ixy="${0.461719*scale}" ixz="${40.230606*scale}" iyy="${280.351624*scale}" iyz="${-1.692201*scale}" izz="${114.922241*scale}"/>
+        <mass value="${m1}"/>
+        <inertia ixx="${256.757294*scale*m1}" ixy="${0.461719*scale*m1}" ixz="${40.230606*scale*m1}" iyy="${280.351624*scale*m1}" iyz="${-1.692201*scale*m1}" izz="${114.922241*scale*m1}"/>
       </inertial>
       <collision name="collision">
@@ -50,6 +64,6 @@
       <inertial>
         <origin xyz="0 0.0371 -0.0015" rpy="0 0 0"/>
-        <mass value="${73.212067 * const}"/>
-        <inertia ixx="${308.272949*scale}" ixy="0" ixz="0" iyy="${141.348206*scale}" iyz="${-6.197227*scale}" izz="${320.700867*scale}"/>
+        <mass value="${m2}"/>
+        <inertia ixx="${308.272949*scale*m2}" ixy="0" ixz="0" iyy="${141.348206*scale*m2}" iyz="${-6.197227*scale*m2}" izz="${320.700867*scale*m2}"/>
       </inertial>
       <collision name="collision">
@@ -70,6 +84,6 @@
       <inertial>
         <origin xyz=" 0 -0.0041 -0.0371" rpy="0 0 0"/>
-        <mass value="${43.109013  * const}"/>
-        <inertia ixx="${177.687561*scale}" ixy="0" ixz="0" iyy="${208.616043*scale}" iyz="${-14.718610*scale}" izz="${59.618698*scale}"/>
+        <mass value="${m3}"/>
+        <inertia ixx="${177.687561*scale*m3}" ixy="0" ixz="0" iyy="${208.616043*scale*m3}" iyz="${-14.718610*scale*m3}" izz="${59.618698*scale*m3}"/>
       </inertial>
       <collision name="collision">
@@ -90,6 +104,6 @@
       <inertial>
         <origin xyz="0.0002  -0.0233 -0.0124" rpy="0 0 0"/>
-        <mass value="${79.043472 * const}"/>
-        <inertia ixx="${609.197083*scale}" ixy="${13.511174*scale}" ixz="${-5.220560*scale}" iyy="${234.447556*scale}" iyz="${179.840118*scale}" izz="${511.354614*scale}"/>
+        <mass value="${m4}"/>
+        <inertia ixx="${609.197083*scale*m4}" ixy="${13.511174*scale*m4}" ixz="${-5.220560*scale*m4}" iyy="${234.447556*scale*m4}" iyz="${179.840118*scale*m4}" izz="${511.354614*scale*m4}"/>
       </inertial>
       <collision name="collision">
@@ -110,8 +124,16 @@
       <inertial>
         <origin xyz="-0.0006 -0.0009 -0.0311" rpy="0 0 0"/>
-        <mass value="${65.552696 * const}"/>
-        <inertia ixx="${385.638153*scale}" ixy="${-0.223889*scale}" ixz="${-13.452513*scale}" iyy="${286.320038*scale}" iyz="${-3.575976*scale}" izz="${338.489807*scale}"/>
-      </inertial>
-      <collision name="collision">
+        <mass value="${m5}"/>
+        <inertia ixx="${385.638153*scale*m5}" ixy="${-0.223889*scale*m5}" ixz="${-13.452513*scale*m5}" iyy="${286.320038*scale*m5}" iyz="${-3.575976*scale*m5}" izz="${338.489807*scale*m5}"/>
+      </inertial>
+      <collision name="collision">
+        <surface>
+			<friction>
+				<ode>
+					<mu>100</mu>
+					<mu2>10</mu2>
+				</ode>
+			</friction>
+		</surface>
         <origin xyz="-0.0006 -0.0009 -0.0311" rpy="0 0 0"/>
         <geometry>
@@ -125,5 +147,5 @@
         </geometry>
       </visual>
-    </link>
+    </link> <!-- -->
     <joint type="fixed" name="leg${suffix}joint0">
       <child link="leg${suffix}link0"/>
@@ -139,5 +161,5 @@
       <limit lower="-1.57" upper="1.57" effort="100" velocity="10"/>
     </joint>
-    <joint type="revolute" name="leg${suffix}joint2">
+     <joint type="revolute" name="leg${suffix}joint2">
       <origin xyz="-0.0309 0.0002 0.0381" rpy="${3.14159/2} 0 ${3.14159 * flipped}"/>
       <child link="leg${suffix}link2"/>
@@ -166,5 +188,5 @@
       <axis xyz="0 1 0"/>
       <limit lower="-1.57" upper="1.57" effort="100" velocity="10"/>
-    </joint>
+    </joint> <!-- -->
 <transmission name="tran1">
     <type>transmission_interface/SimpleTransmission</type>
