Commit message: simulation working, alpha interplation working, getting data

File: src/daedalus_description/urdf/daedalus.urdf (robot description, URDF)
Before this commit: robot daedalus, 8 links, 7 joints
Links:
- removed link chasis
- removed link world
- added link frame, mass 2.40264202; collision box size=0.28 0.125 0.06; visual box size=0.28 0.125 0.06
- added link leg2link0, mass 0.47264202; collision mesh filename=package://daedalus_description/meshes/link0.dae; visual mesh filename=package://daedalus_description/meshes/link0.dae
- added link leg2link1, mass 0.62343552; collision mesh filename=package://daedalus_description/meshes/link1.dae; visual mesh filename=package://daedalus_description/meshes/link1.dae
- added link leg2link2, mass 0.73212067; collision mesh filename=package://daedalus_description/meshes/link2.dae; visual mesh filename=package://daedalus_description/meshes/link2.dae
- added link leg2link3, mass 0.43109013; collision mesh filename=package://daedalus_description/meshes/link3.dae; visual mesh filename=package://daedalus_description/meshes/link3.dae
- added link leg2link4, mass 0.79043472; collision mesh filename=package://daedalus_description/meshes/link4.dae; visual mesh filename=package://daedalus_description/meshes/link4.dae
- added link leg2link5, mass 0.65552696; collision mesh filename=package://daedalus_description/meshes/link5.dae; visual mesh filename=package://daedalus_description/meshes/link5.dae
- added link leg3link0, mass 0.47264202; collision mesh filename=package://daedalus_description/meshes/link0.dae; visual mesh filename=package://daedalus_description/meshes/link0.dae
- added link leg3link1, mass 0.62343552; collision mesh filename=package://daedalus_description/meshes/link1.dae; visual mesh filename=package://daedalus_description/meshes/link1.dae
- added link leg3link2, mass 0.73212067; collision mesh filename=package://daedalus_description/meshes/link2.dae; visual mesh filename=package://daedalus_description/meshes/link2.dae
- added link leg3link3, mass 0.43109013; collision mesh filename=package://daedalus_description/meshes/link3.dae; visual mesh filename=package://daedalus_description/meshes/link3.dae
- added link leg3link4, mass 0.79043472; collision mesh filename=package://daedalus_description/meshes/link4.dae; visual mesh filename=package://daedalus_description/meshes/link4.dae
- added link leg3link5, mass 0.65552696; collision mesh filename=package://daedalus_description/meshes/link5.dae; visual mesh filename=package://daedalus_description/meshes/link5.dae
- added link leg4link0, mass 0.47264202; collision mesh filename=package://daedalus_description/meshes/link0.dae; visual mesh filename=package://daedalus_description/meshes/link0.dae
- added link leg4link1, mass 0.62343552; collision mesh filename=package://daedalus_description/meshes/link1.dae; visual mesh filename=package://daedalus_description/meshes/link1.dae
- added link leg4link2, mass 0.73212067; collision mesh filename=package://daedalus_description/meshes/link2.dae; visual mesh filename=package://daedalus_description/meshes/link2.dae
- added link leg4link3, mass 0.43109013; collision mesh filename=package://daedalus_description/meshes/link3.dae; visual mesh filename=package://daedalus_description/meshes/link3.dae
- added link leg4link4, mass 0.79043472; collision mesh filename=package://daedalus_description/meshes/link4.dae; visual mesh filename=package://daedalus_description/meshes/link4.dae
- added link leg4link5, mass 0.65552696; collision mesh filename=package://daedalus_description/meshes/link5.dae; visual mesh filename=package://daedalus_description/meshes/link5.dae
- added link root
- link leg1link0: mass 0.472639954 -> 0.47264202
- link leg1link1: mass 0.623121787 -> 0.62343552
- link leg1link2: mass 0.732147232 -> 0.73212067
- link leg1link3: mass 0.431132052 -> 0.43109013
- link leg1link4: mass 0.790197358 -> 0.79043472
- link leg1link5: mass 0.655679875 -> 0.65552696
Joints:
- removed joint base
- added joint leg2joint0: type fixed, parent frame, child leg2link0, origin xyz=0.14 -0.0625 0 rpy=0 0 3.14, axis 1 0 0
- added joint leg2joint1: type revolute, parent leg2link0, child leg2link1, origin xyz=-0.0249 0 0.0205 rpy=0 0 0, axis 0 0 -1, limit lower=-1.57 upper=1.57 effort=100 velocity=10
- added joint leg2joint2: type revolute, parent leg2link1, child leg2link2, origin xyz=-0.0309 0.0002 0.0381 rpy=1.570795 0 0.0, axis 1.0 0 0, limit lower=-1.57 upper=1.57 effort=100 velocity=10
- added joint leg2joint3: type revolute, parent leg2link2, child leg2link3, origin xyz=0 0.0564 -0.0208 rpy=0 0 0, axis -1.0 0 0, limit lower=-1.57 upper=1.57 effort=100 velocity=10
- added joint leg2joint4: type revolute, parent leg2link3, child leg2link4, origin xyz=0 -0.0171 -0.0742 rpy=-0.7853975 0 0, axis -1.0 0 0, limit lower=-1.57 upper=1.57 effort=100 velocity=10
- added joint leg2joint5: type revolute, parent leg2link4, child leg2link5, origin xyz=-0.0004 -0.0411 -0.0248 rpy=0 0 0, axis 0 1 0, limit lower=-1.57 upper=1.57 effort=100 velocity=10
- added joint leg3joint0: type fixed, parent frame, child leg3link0, origin xyz=-0.14 0.0625 0 rpy=0 0 0, axis 1 0 0
- added joint leg3joint1: type revolute, parent leg3link0, child leg3link1, origin xyz=-0.0249 0 0.0205 rpy=0 0 0, axis 0 0 -1, limit lower=-1.57 upper=1.57 effort=100 velocity=10
- added joint leg3joint2: type revolute, parent leg3link1, child leg3link2, origin xyz=-0.0309 0.0002 0.0381 rpy=1.570795 0 0.0, axis 1.0 0 0, limit lower=-1.57 upper=1.57 effort=100 velocity=10
- added joint leg3joint3: type revolute, parent leg3link2, child leg3link3, origin xyz=0 0.0564 -0.0208 rpy=0 0 0, axis -1.0 0 0, limit lower=-1.57 upper=1.57 effort=100 velocity=10
- added joint leg3joint4: type revolute, parent leg3link3, child leg3link4, origin xyz=0 -0.0171 -0.0742 rpy=-0.7853975 0 0, axis -1.0 0 0, limit lower=-1.57 upper=1.57 effort=100 velocity=10
- added joint leg3joint5: type revolute, parent leg3link4, child leg3link5, origin xyz=-0.0004 -0.0411 -0.0248 rpy=0 0 0, axis 0 1 0, limit lower=-1.57 upper=1.57 effort=100 velocity=10
- added joint leg4joint0: type fixed, parent frame, child leg4link0, origin xyz=-0.14 -0.0625 0 rpy=0 0 0, axis 1 0 0
- added joint leg4joint1: type revolute, parent leg4link0, child leg4link1, origin xyz=-0.0249 0 0.0205 rpy=0 0 0, axis 0 0 -1, limit lower=-1.57 upper=1.57 effort=100 velocity=10
- added joint leg4joint2: type revolute, parent leg4link1, child leg4link2, origin xyz=-0.0309 0.0002 0.0381 rpy=1.570795 0 3.14159, axis -1.0 0 0, limit lower=-1.57 upper=1.57 effort=100 velocity=10
- added joint leg4joint3: type revolute, parent leg4link2, child leg4link3, origin xyz=0 0.0564 -0.0208 rpy=0 0 0, axis 1.0 0 0, limit lower=-1.57 upper=1.57 effort=100 velocity=10
- added joint leg4joint4: type revolute, parent leg4link3, child leg4link4, origin xyz=0 -0.0171 -0.0742 rpy=-0.7853975 0 0, axis 1.0 0 0, limit lower=-1.57 upper=1.57 effort=100 velocity=10
- added joint leg4joint5: type revolute, parent leg4link4, child leg4link5, origin xyz=-0.0004 -0.0411 -0.0248 rpy=0 0 0, axis 0 1 0, limit lower=-1.57 upper=1.57 effort=100 velocity=10
- added joint r_root: type fixed, parent root, child frame
- joint leg1joint0: origin xyz=-1.035 -1.125 0 rpy=0 0 0 -> xyz=0.14 0.0625 0 rpy=0 0 3.14; parent chasis -> frame
- joint leg1joint1: axis 0 0 1 -> 0 0 -1; limit lower=-1.57 upper=1.57 effort=100 velocity=0.5 -> lower=-1.57 upper=1.57 effort=100 velocity=10; origin xyz=0.86 1.03 0.17 rpy=0 0 0 -> xyz=-0.0249 0 0.0205 rpy=0 0 0
- joint leg1joint2: axis 1 0 0 -> -1.0 0 0; limit lower=-0.45 upper=3.59 effort=100 velocity=0.5 -> lower=-1.57 upper=1.57 effort=100 velocity=10; origin xyz=-0.01 0 0.04 rpy=0 0 0 -> xyz=-0.0309 0.0002 0.0381 rpy=1.570795 0 3.14159
- joint leg1joint3: axis 1 0 0 -> 1.0 0 0; limit lower=-1.57 upper=1.57 effort=100 velocity=0.5 -> lower=-1.57 upper=1.57 effort=100 velocity=10; origin xyz=0 0.06 -0.02 rpy=0 0 0 -> xyz=0 0.0564 -0.0208 rpy=0 0 0
- joint leg1joint4: axis 1 0 0 -> 1.0 0 0; limit lower=-1.57 upper=1.57 effort=100 velocity=0.5 -> lower=-1.57 upper=1.57 effort=100 velocity=10; origin xyz=-0.04 -0.02 -0.08 rpy=0 0 0 -> xyz=0 -0.0171 -0.0742 rpy=-0.7853975 0 0
- joint leg1joint5: limit lower=-1.57 upper=1.57 effort=100 velocity=0.5 -> lower=-1.57 upper=1.57 effort=100 velocity=10; origin xyz=0.02 -0.04 -0.02 rpy=0 0 0 -> xyz=-0.0004 -0.0411 -0.0248 rpy=0 0 0
